File: trunk/Schematics/bt-lights.brd (EAGLE design)
At the start: 104.1 x 73.1 mm, 25 parts, among them IC1 MAX6966

Commit message: ADDED:  - the world famous icon  - new protocol revision  - schematics and layout (prelim)
Parts:
- added R11: 10k, resistor:0207/7
Connections:
- net AT: now also R11.2
- net GND: now also R11.1
Routing:
- net GND: track 116.5 -> 128.7 mm
- net AT: track 43.1 -> 52.1 mm
Changed lines of the file:
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@@
 <element name="R9" library="resistor" package="0207/7" value="1k" x="86.36" y="40.132" rot="R90"/>
 <element name="R10" library="resistor" package="0207/7" value="1k" x="96.52" y="40.132" rot="R90"/>
+<element name="R11" library="resistor" package="0207/7" value="10k" x="25.146" y="9.906"/>
 </elements>
 <signals>
@@
 <wire x1="60.96" y1="7.239" x2="60.96" y2="7.112" width="0.254" layer="1"/>
 <wire x1="18.288" y1="11.811" x2="18.03" y2="11.942" width="0.254" layer="1"/>
+<contactref element="R11" pad="1"/>
+<wire x1="21.336" y1="9.906" x2="9.83" y2="9.906" width="0.4064" layer="16"/>
+<wire x1="9.83" y1="9.906" x2="9.83" y2="9.142" width="0.4064" layer="16"/>
+<wire x1="9.83" y1="9.142" x2="9.83" y2="9.142" width="0" layer="19" extent="1-16"/>
 </signal>
 <signal name="+5V">
@@
 <contactref element="BT_INTERFACE" pad="34"/>
 <wire x1="9.906" y1="26.289" x2="9.906" y2="27.813" width="0.254" layer="1"/>
-<wire x1="27.432" y1="8.763" x2="9.906" y2="26.289" width="0.254" layer="16"/>
-<wire x1="41.529" y1="8.763" x2="27.432" y2="8.763" width="0.254" layer="16"/>
-<wire x1="43.18" y1="7.112" x2="41.529" y2="8.763" width="0.254" layer="16"/>
+<wire x1="28.956" y1="9.906" x2="28.956" y2="14.478" width="0.254" layer="16"/>
+<wire x1="28.956" y1="14.478" x2="12.192" y2="14.478" width="0.254" layer="16"/>
+<wire x1="12.192" y1="14.478" x2="12.192" y2="23.622" width="0.254" layer="16"/>
+<wire x1="12.192" y1="23.622" x2="9.906" y2="26.289" width="0.254" layer="16"/>
 <wire x1="9.906" y1="27.813" x2="9.53" y2="27.942" width="0.254" layer="1"/>
 <via x="9.906" y="26.289" extent="1-16" drill="0.6096"/>
+<contactref element="R11" pad="2"/>
+<wire x1="28.956" y1="9.906" x2="41.148" y2="9.906" width="0.4064" layer="16"/>
+<wire x1="41.148" y1="9.906" x2="42.672" y2="8.382" width="0.4064" layer="16"/>
+<wire x1="42.672" y1="8.382" x2="42.672" y2="7.62" width="0.4064" layer="16"/>
+<wire x1="42.672" y1="7.62" x2="43.434" y2="6.858" width="0.4064" layer="16"/>
+<wire x1="43.434" y1="6.858" x2="43.18" y2="7.112" width="0" layer="19" extent="1-16"/>
 </signal>
 <signal name="RX">

Commit message: UPDATE:  - new hardware fix in schematic  - new commands in test gui  - new pinning documented ADDED:  - NETDUINO schematic
Parts:
- added FREQ_SELECTOR: (no value), con-lstb:MA03-1
- MCU_CONNECTOR: device con-lsta:FE10 -> con-lsta:FE15
Connections:
- new net N$15: FREQ_SELECTOR.3, MCU_CONNECTOR.11
- new net N$16: FREQ_SELECTOR.2, IC1.14
- net +3V3: now also MCU_CONNECTOR.8; no longer MCU_CONNECTOR.3
- net +5V: now also MCU_CONNECTOR.9; no longer MCU_CONNECTOR.2
- net AT: now also MCU_CONNECTOR.3; no longer MCU_CONNECTOR.8
- net GND: now also MCU_CONNECTOR.10; no longer MCU_CONNECTOR.1
- net N$1: now also MCU_CONNECTOR.7; no longer MCU_CONNECTOR.4
- net N$2: now also MCU_CONNECTOR.4; no longer MCU_CONNECTOR.7
- net N$3: now also MCU_CONNECTOR.6; no longer MCU_CONNECTOR.5
- net N$4: now also FREQ_SELECTOR.1, MCU_CONNECTOR.5; no longer IC1.14, MCU_CONNECTOR.6
- net RX: now also MCU_CONNECTOR.2; no longer MCU_CONNECTOR.9
- net TX: now also MCU_CONNECTOR.1; no longer MCU_CONNECTOR.10
Routing:
- net N$4: track 46.3 -> 0.00 mm, vias 1 -> 0
- net N$16: track 0.00 -> 46.0 mm, vias 0 -> 1
- net N$1: track 44.8 -> 42.0 mm
- net GND: track 128.7 -> 126.6 mm
- net +3V3: track 96.2 -> 94.4 mm
- net +5V: track 168.3 -> 166.7 mm
