File: trunk/Schematics/bt-lights-shield.sch (EAGLE design)
At the start: 27 parts, among them IC1 MAX6966, U1 ARDUINO_SHIELDNO_SILK

Commit message: Update App for setup view
Parts:
- removed EL_CONNECTOR: (no value), con-lstb:MA20-1L
- added JP1, JP10, JP2, JP3, JP4, JP5, JP6, JP7, JP8, JP9: (no value), SparkFun-Connectors:M02-JST-2MM-SMT
- HIGHVOLTAGE: device pinhead:PINHD-1X2 -> SparkFun-Connectors:M02-JST-2MM-SMT
Connections:
- net N$P1 renamed IN1
- net N$P2 renamed IN2
- net N$P3 renamed IN3
- net N$P4 renamed IN4
- net N$P5 renamed IN5
- net N$P6 renamed IN6
- net N$P7 renamed IN7
- net N$P8 renamed IN8
- net N$P9 renamed IN9
- net OUT0: now also JP1.2; no longer EL_CONNECTOR.1
- net OUT1: now also JP2.2; no longer EL_CONNECTOR.3
- net OUT2: now also JP3.2; no longer EL_CONNECTOR.5
- net OUT3: now also JP4.2; no longer EL_CONNECTOR.7
- net OUT4: now also JP5.2; no longer EL_CONNECTOR.9
- net OUT5: now also JP6.2; no longer EL_CONNECTOR.11
- net OUT6: now also JP7.2; no longer EL_CONNECTOR.13
- net OUT7: now also JP8.2; no longer EL_CONNECTOR.15
- net OUT8: now also JP9.2; no longer EL_CONNECTOR.17
- net OUT9: now also JP10.2; no longer EL_CONNECTOR.19
- net VDD: now also JP1.1, JP10.1, JP2.1, JP3.1, JP4.1, JP5.1, JP6.1, JP7.1, JP8.1, JP9.1; no longer EL_CONNECTOR.10, EL_CONNECTOR.12, EL_CONNECTOR.14, EL_CONNECTOR.16, EL_CONNECTOR.18, EL_CONNECTOR.2, EL_CONNECTOR.20, EL_CONNECTOR.4, EL_CONNECTOR.6, EL_CONNECTOR.8
Other:
- moved on the sheet: HIGHVOLTAGE
